Commit message: Update to xarm_ros2 jazzy 3dc2b5e (xarm_sdk v1.18.1)
Unmodified upstream xArm-Developer/xarm_ros2 jazzy branch, SDK submodule
included as plain files. This is the version built and tested with the
Lite6 on ROS 2 Jazzy.

Co-Authored-By: Claude Opus 5.5 <noreply@anthropic.com>

File: xarm_description/urdf/dual_xarm_device.urdf.xacro (robot description, xacro)
@@ -25,4 +25,8 @@
   <xacro:arg name="report_type_1" default="normal"/>
   <xacro:arg name="report_type_2" default="normal"/>
+  <xacro:arg name="attach_xyz_1" default="0 0 0"/>
+  <xacro:arg name="attach_rpy_1" default="0 0 0"/>
+  <xacro:arg name="attach_xyz_2" default="0 1 0"/>
+  <xacro:arg name="attach_rpy_2" default="0 0 0"/>
   <xacro:arg name="ros2_control_plugin" default="uf_robot_hardware/UFRobotSystemHardware"/>
   <xacro:arg name="ros2_control_params" default=""/>
@@ -62,4 +66,6 @@
   <xacro:arg name="kinematics_suffix_1" default=""/>
   <xacro:arg name="kinematics_suffix_2" default=""/>
+  <xacro:arg name="gripper_version_1" default="G1"/>
+  <xacro:arg name="gripper_version_2" default="G1"/>
   <!-- load xarm device -->
   <xacro:include filename="$(find xarm_description)/urdf/xarm_device_macro.xacro" />
@@ -70,5 +76,5 @@
     ros2_control_plugin="$(arg ros2_control_plugin)" robot_type="$(arg robot_type_1)"
     load_gazebo_plugin="false" ros2_control_params="$(arg ros2_control_params)"
-    attach_to="world" attach_xyz="0 0 0" attach_rpy="0 0 0"
+    attach_to="world" attach_xyz="$(arg attach_xyz_1)" attach_rpy="$(arg attach_rpy_1)"
     add_realsense_d435i="$(arg add_realsense_d435i_1)"
     add_d435i_links="$(arg add_d435i_links_1)"
@@ -82,5 +88,5 @@
     robot_ip="$(arg robot_ip_1)" report_type="$(arg report_type_1)"
     baud_checkset="$(arg baud_checkset_1)" default_gripper_baud="$(arg default_gripper_baud_1)"
-    model1300="$(arg model1300_1)" robot_sn="$(arg robot_sn_1)" mesh_suffix="$(arg mesh_suffix)" kinematics_suffix="$(arg kinematics_suffix_1)" />
+    model1300="$(arg model1300_1)" robot_sn="$(arg robot_sn_1)" mesh_suffix="$(arg mesh_suffix)" kinematics_suffix="$(arg kinematics_suffix_1)" gripper_version="$(arg gripper_version_1)" />
   <xacro:xarm_device prefix="$(arg prefix_2)" hw_ns="$(arg hw_ns)" limited="$(arg limited)"
     effort_control="$(arg effort_control)" velocity_control="$(arg velocity_control)"
@@ -89,5 +95,5 @@
     ros2_control_plugin="$(arg ros2_control_plugin)" robot_type="$(arg robot_type_2)"
     load_gazebo_plugin="true" ros2_control_params="$(arg ros2_control_params)"
-    attach_to="world" attach_xyz="0 1 0" attach_rpy="0 0 0" create_attach_link="false"
+    attach_to="world" attach_xyz="$(arg attach_xyz_2)" attach_rpy="$(arg attach_rpy_2)" create_attach_link="false"
     add_realsense_d435i="$(arg add_realsense_d435i_2)"
     add_d435i_links="$(arg add_d435i_links_2)"
@@ -101,4 +107,4 @@
     robot_ip="$(arg robot_ip_2)" report_type="$(arg report_type_2)"
     baud_checkset="$(arg baud_checkset_2)" default_gripper_baud="$(arg default_gripper_baud_2)"
-    model1300="$(arg model1300_2)" robot_sn="$(arg robot_sn_2)" mesh_suffix="$(arg mesh_suffix)" kinematics_suffix="$(arg kinematics_suffix_2)" />
+    model1300="$(arg model1300_2)" robot_sn="$(arg robot_sn_2)" mesh_suffix="$(arg mesh_suffix)" kinematics_suffix="$(arg kinematics_suffix_2)" gripper_version="$(arg gripper_version_2)" />
 </robot>

File: xarm_description/urdf/gripper/bio_gripper.urdf.xacro (robot description, xacro)
@@ -1,5 +1,13 @@
 <?xml version="1.0"?>
 <robot xmlns:xacro="http://ros.org/wiki/xacro" name="uf_bio_gripper">
-  <xacro:macro name="bio_gripper_urdf" params="prefix:='' attach_to:='' attach_xyz:='0 0 0' attach_rpy:='0 0 0' ">
+  <xacro:macro name="bio_gripper_urdf" params="prefix:='' attach_to:='' attach_xyz:='0 0 0' attach_rpy:='0 0 0' gripper_version:='G1' ">
+    <xacro:property name="add_mesh_suffix" value="true"/>
+    <xacro:property name="other_mesh_suffix" value=""/>
+    <xacro:property name="name_suffix" value=""/>
+    <xacro:if value="${gripper_version == 'G2' or gripper_version == 'g2'}">
+      <xacro:property name="name_suffix" value="_g2"/>
+      <xacro:property name="other_mesh_suffix" value="dae"/>
+      <xacro:property name="add_mesh_suffix" value="false"/>
+    </xacro:if>
     <xacro:unless value="${attach_to == ''}">
       <joint name="${prefix}bio_gripper_fix" type="fixed">
@@ -18,10 +26,14 @@
       </inertial>
       <xacro:common_link_visual
-        mesh_filename="gripper/bio/link_base"
+        mesh_filename="gripper/bio/link_base${name_suffix}"
+        add_mesh_suffix="${add_mesh_suffix}"
+        other_mesh_suffix="${other_mesh_suffix}"
         origin_xyz="0 0 0"
         origin_rpy="0 0 0"
         material_name="${prefix}White" />
       <xacro:common_link_collision
-        mesh_filename="gripper/bio/link_base"
+        mesh_filename="gripper/bio/link_base${name_suffix}"
+        add_mesh_suffix="${add_mesh_suffix}"
+        other_mesh_suffix="${other_mesh_suffix}"
         origin_xyz="0 0 0"
         origin_rpy="0 0 0" />
@@ -36,10 +48,14 @@
       </inertial>
       <xacro:common_link_visual
-        mesh_filename="gripper/bio/left_finger"
+        mesh_filename="gripper/bio/left_finger${name_suffix}"
+        add_mesh_suffix="${add_mesh_suffix}"
+        other_mesh_suffix="${other_mesh_suffix}"
         origin_xyz="0 0 0"
         origin_rpy="0 0 0"
         material_name="${prefix}White" />
       <xacro:common_link_collision
-        mesh_filename="gripper/bio/left_finger"
+        mesh_filename="gripper/bio/left_finger${name_suffix}"
+        add_mesh_suffix="${add_mesh_suffix}"
+        other_mesh_suffix="${other_mesh_suffix}"
         origin_xyz="0 0 0"
         origin_rpy="0 0 0" />
@@ -62,10 +78,14 @@
       </inertial>
       <xacro:common_link_visual
-        mesh_filename="gripper/bio/right_finger"
+        mesh_filename="gripper/bio/right_finger${name_suffix}"
+        add_mesh_suffix="${add_mesh_suffix}"
+        other_mesh_suffix="${other_mesh_suffix}"
         origin_xyz="0 0 0"
         origin_rpy="0 0 0"
         material_name="${prefix}White" />
       <xacro:common_link_collision
-        mesh_filename="gripper/bio/right_finger"
+        mesh_filename="gripper/bio/right_finger${name_suffix}"
+        add_mesh_suffix="${add_mesh_suffix}"
+        other_mesh_suffix="${other_mesh_suffix}"
         origin_xyz="0 0 0"
         origin_rpy="0 0 0" />

File: xarm_description/urdf/gripper/xarm_gripper.urdf.xacro (robot description, xacro)
@@ -1,5 +1,13 @@
 <?xml version="1.0"?>
 <robot xmlns:xacro="http://ros.org/wiki/xacro" name="xarm_gripper">
-  <xacro:macro name="xarm_gripper_urdf" params="prefix:='' attach_to:='' attach_xyz:='0 0 0' attach_rpy:='0 0 0' ">
+  <xacro:macro name="xarm_gripper_urdf" params="prefix:='' attach_to:='' attach_xyz:='0 0 0' attach_rpy:='0 0 0' gripper_version:='G1' ">
+    <xacro:property name="add_mesh_suffix" value="true"/>
+    <xacro:property name="other_mesh_suffix" value=""/>
+    <xacro:property name="name_suffix" value=""/>
+    <xacro:if value="${gripper_version == 'G2' or gripper_version == 'g2'}">
+      <xacro:property name="name_suffix" value="_g2"/>
+      <xacro:property name="other_mesh_suffix" value="dae"/>
+      <xacro:property name="add_mesh_suffix" value="false"/>
+    </xacro:if>
     <xacro:unless value="${attach_to == ''}">
       <joint name="${prefix}gripper_fix" type="fixed">
@@ -18,10 +26,14 @@
       </inertial>
       <xacro:common_link_visual
-        mesh_filename="gripper/xarm/base_link"
+        mesh_filename="gripper/xarm/base_link${name_suffix}"
+        add_mesh_suffix="${add_mesh_suffix}"
+        other_mesh_suffix="${other_mesh_suffix}"
         origin_xyz="0 0 0"
         origin_rpy="0 0 0"
         material_name="${prefix}White" />
       <xacro:common_link_collision
-        mesh_filename="gripper/xarm/base_link"
+        mesh_filename="gripper/xarm/base_link${name_suffix}"
+        add_mesh_suffix="${add_mesh_suffix}"
+        other_mesh_suffix="${other_mesh_suffix}"
         origin_xyz="0 0 0"
         origin_rpy="0 0 0" />
@@ -36,10 +48,14 @@
       </inertial>
       <xacro:common_link_visual
-        mesh_filename="gripper/xarm/left_outer_knuckle"
-        origin_xyz="0 0 0"
-        origin_rpy="0 0 0"
-        material_name="${prefix}Silver" />
-      <xacro:common_link_collision
-        mesh_filename="gripper/xarm/left_outer_knuckle"
+        mesh_filename="gripper/xarm/left_outer_knuckle${name_suffix}"
+        add_mesh_suffix="${add_mesh_suffix}"
+        other_mesh_suffix="${other_mesh_suffix}"
+        origin_xyz="0 0 0"
+        origin_rpy="0 0 0"
+        material_name="${prefix}Silver" />
+      <xacro:common_link_collision
+        mesh_filename="gripper/xarm/left_outer_knuckle${name_suffix}"
+        add_mesh_suffix="${add_mesh_suffix}"
+        other_mesh_suffix="${other_mesh_suffix}"
         origin_xyz="0 0 0"
         origin_rpy="0 0 0" />
@@ -61,10 +77,14 @@
       </inertial>
       <xacro:common_link_visual
-        mesh_filename="gripper/xarm/left_finger"
-        origin_xyz="0 0 0"
-        origin_rpy="0 0 0"
-        material_name="${prefix}Silver" />
-      <xacro:common_link_collision
-        mesh_filename="gripper/xarm/left_finger"
+        mesh_filename="gripper/xarm/left_finger${name_suffix}"
+        add_mesh_suffix="${add_mesh_suffix}"
+        other_mesh_suffix="${other_mesh_suffix}"
+        origin_xyz="0 0 0"
+        origin_rpy="0 0 0"
+        material_name="${prefix}Silver" />
+      <xacro:common_link_collision
+        mesh_filename="gripper/xarm/left_finger${name_suffix}"
+        add_mesh_suffix="${add_mesh_suffix}"
+        other_mesh_suffix="${other_mesh_suffix}"
         origin_xyz="0 0 0"
         origin_rpy="0 0 0" />
@@ -87,10 +107,14 @@
       </inertial>
       <xacro:common_link_visual
-        mesh_filename="gripper/xarm/left_inner_knuckle"
-        origin_xyz="0 0 0"
-        origin_rpy="0 0 0"
-        material_name="${prefix}Silver" />
-      <xacro:common_link_collision
-        mesh_filename="gripper/xarm/left_inner_knuckle"
+        mesh_filename="gripper/xarm/left_inner_knuckle${name_suffix}"
+        add_mesh_suffix="${add_mesh_suffix}"
+        other_mesh_suffix="${other_mesh_suffix}"
+        origin_xyz="0 0 0"
+        origin_rpy="0 0 0"
+        material_name="${prefix}Silver" />
+      <xacro:common_link_collision
+        mesh_filename="gripper/xarm/left_inner_knuckle${name_suffix}"
+        add_mesh_suffix="${add_mesh_suffix}"
+        other_mesh_suffix="${other_mesh_suffix}"
         origin_xyz="0 0 0"
         origin_rpy="0 0 0" />
@@ -113,10 +137,14 @@
       </inertial>
       <xacro:common_link_visual
-        mesh_filename="gripper/xarm/right_outer_knuckle"
-        origin_xyz="0 0 0"
-        origin_rpy="0 0 0"
-        material_name="${prefix}Silver" />
-      <xacro:common_link_collision
-        mesh_filename="gripper/xarm/right_outer_knuckle"
+        mesh_filename="gripper/xarm/right_outer_knuckle${name_suffix}"
+        add_mesh_suffix="${add_mesh_suffix}"
+        other_mesh_suffix="${other_mesh_suffix}"
+        origin_xyz="0 0 0"
+        origin_rpy="0 0 0"
+        material_name="${prefix}Silver" />
+      <xacro:common_link_collision
+        mesh_filename="gripper/xarm/right_outer_knuckle${name_suffix}"
+        add_mesh_suffix="${add_mesh_suffix}"
+        other_mesh_suffix="${other_mesh_suffix}"
         origin_xyz="0 0 0"
         origin_rpy="0 0 0" />
@@ -139,10 +167,14 @@
       </inertial>
       <xacro:common_link_visual
-        mesh_filename="gripper/xarm/right_finger"
-        origin_xyz="0 0 0"
-        origin_rpy="0 0 0"
-        material_name="${prefix}Silver" />
-      <xacro:common_link_collision
-        mesh_filename="gripper/xarm/right_finger"
+        mesh_filename="gripper/xarm/right_finger${name_suffix}"
+        add_mesh_suffix="${add_mesh_suffix}"
+        other_mesh_suffix="${other_mesh_suffix}"
+        origin_xyz="0 0 0"
+        origin_rpy="0 0 0"
+        material_name="${prefix}Silver" />
+      <xacro:common_link_collision
+        mesh_filename="gripper/xarm/right_finger${name_suffix}"
+        add_mesh_suffix="${add_mesh_suffix}"
+        other_mesh_suffix="${other_mesh_suffix}"
         origin_xyz="0 0 0"
         origin_rpy="0 0 0" />
@@ -165,10 +197,14 @@
       </inertial>
       <xacro:common_link_visual
-        mesh_filename="gripper/xarm/right_inner_knuckle"
-        origin_xyz="0 0 0"
-        origin_rpy="0 0 0"
-        material_name="${prefix}Silver" />
-      <xacro:common_link_collision
-        mesh_filename="gripper/xarm/right_inner_knuckle"
+        mesh_filename="gripper/xarm/right_inner_knuckle${name_suffix}"
+        add_mesh_suffix="${add_mesh_suffix}"
+        other_mesh_suffix="${other_mesh_suffix}"
+        origin_xyz="0 0 0"
+        origin_rpy="0 0 0"
+        material_name="${prefix}Silver" />
+      <xacro:common_link_collision
+        mesh_filename="gripper/xarm/right_inner_knuckle${name_suffix}"
+        add_mesh_suffix="${add_mesh_suffix}"
+        other_mesh_suffix="${other_mesh_suffix}"
         origin_xyz="0 0 0"
         origin_rpy="0 0 0" />

File: xarm_description/urdf/xarm_device.urdf.xacro (robot description, xacro)
@@ -9,5 +9,4 @@
   <xacro:arg name="add_vacuum_gripper" default="false"/>
   <xacro:arg name="add_bio_gripper" default="false"/>
-  <xacro:arg name="add_robotiq_arg85" default="false"/>
   <xacro:arg name="model1300" default="false"/>
   <xacro:arg name="dof" default="7"/>
@@ -40,4 +39,5 @@
   <xacro:arg name="mesh_suffix" default="stl"/>
   <xacro:arg name="kinematics_suffix" default=""/>
+  <xacro:arg name="gripper_version" default="G1"/>
   <!-- load xarm device -->
   <xacro:include filename="$(find xarm_description)/urdf/xarm_device_macro.xacro" />
@@ -45,5 +45,5 @@
     effort_control="$(arg effort_control)" velocity_control="$(arg velocity_control)"
     add_gripper="$(arg add_gripper)" add_vacuum_gripper="$(arg add_vacuum_gripper)"
-    add_bio_gripper="$(arg add_bio_gripper)" add_robotiq_arg85="$(arg add_robotiq_arg85)" dof="$(arg dof)"
+    add_bio_gripper="$(arg add_bio_gripper)" dof="$(arg dof)"
     ros2_control_plugin="$(arg ros2_control_plugin)" robot_type="$(arg robot_type)"
     load_gazebo_plugin="true" ros2_control_params="$(arg ros2_control_params)"
@@ -60,4 +60,5 @@
     baud_checkset="$(arg baud_checkset)" default_gripper_baud="$(arg default_gripper_baud)"
     model1300="$(arg model1300)" attach_to="$(arg attach_to)" attach_xyz="$(arg attach_xyz)" attach_rpy="$(arg attach_rpy)"
-    robot_sn="$(arg robot_sn)" use_gazebo_camera="$(arg use_gazebo_camera)" mesh_suffix="$(arg mesh_suffix)" kinematics_suffix="$(arg kinematics_suffix)" />
+    robot_sn="$(arg robot_sn)" use_gazebo_camera="$(arg use_gazebo_camera)" mesh_suffix="$(arg mesh_suffix)" kinematics_suffix="$(arg kinematics_suffix)"
+    gripper_version="$(arg gripper_version)" />
 </robot>

File: xarm_description/urdf/xarm_device_macro.xacro (robot description, xacro)
@@ -10,5 +10,4 @@
     add_vacuum_gripper:=false
     add_bio_gripper:=false
-    add_robotiq_arg85:=false
     dof:=7
     robot_type:='xarm'
@@ -43,4 +42,5 @@
     mesh_suffix:='stl'
     kinematics_suffix:=''
+    gripper_version:='G1'
     "
     >
@@ -208,5 +208,18 @@
       <xacro:if value="${add_d435i_links}">
         <xacro:include filename="$(find xarm_description)/urdf/camera/realsense.gazebo.xacro" />
-        <xacro:realsense_gazebo prefix="${prefix}" />
+        <xacro:if value="${is_ros2}">
+          <xacro:if value="${ros2_control_plugin == 'gz_ros2_control/GazeboSimSystem'}">
+            <xacro:realsense_gz prefix="${prefix}" />
+          </xacro:if>
+          <xacro:if value="${ros2_control_plugin == 'ign_ros2_control/IgnitionSystem'}">
+            <xacro:realsense_ignition prefix="${prefix}" />
+          </xacro:if>
+          <xacro:if value="${ros2_control_plugin == 'gazebo_ros2_control/GazeboSystem'}">
+            <xacro:realsense_gazebo prefix="${prefix}" />
+          </xacro:if>
+        </xacro:if>
+        <xacro:unless value="${is_ros2}">
+          <xacro:realsense_gazebo prefix="${prefix}" />
+        </xacro:unless>
       </xacro:if>
     </xacro:if>
@@ -222,6 +235,8 @@
       <xacro:if value="${robot_type == 'lite'}">
         <!-- Load Lite Gripper Model URDF -->
-        <xacro:include filename="$(find xarm_description)/urdf/gripper/lite_gripper.urdf.xacro" />
-        <xacro:uflite_gripper_urdf prefix="${prefix}" attach_to="${prefix}link_eef" />
+        <xacro:include filename="$(find xarm_description)/urdf/gripper/uflite_gripper_macro.xacro" />
+        <xacro:uflite_gripper_macro prefix="${prefix}" attach_to="${prefix}link_eef"
+          ros2_control_plugin="${ros2_control_plugin}" dof="${dof}" hard_interface="${hard_interface}"
+          gripper_version="${gripper_version}" />
       </xacro:if>
       <xacro:unless value="${robot_type == 'lite'}">
@@ -229,22 +244,18 @@
         <xacro:include filename="$(find xarm_description)/urdf/gripper/xarm_gripper_macro.xacro" />
         <xacro:xarm_gripper_macro prefix="${prefix}" attach_to="${prefix}link_eef"
-          ros2_control_plugin="${ros2_control_plugin}" dof="${dof}" hard_interface="${hard_interface}" />
-      </xacro:unless>
-    </xacro:if>
-    <xacro:if value="${not add_gripper and add_robotiq_arg85}">
-      <!-- Load Robotiq arg85 Gripper Model URDF -->
-      <xacro:include filename="$(find xarm_description)/urdf/gripper/robotiq_arg85_macro.xacro" />
-      <xacro:robotiq_arg85_macro prefix="${prefix}" attach_to="${prefix}link_eef"
-        ros2_control_plugin="${ros2_control_plugin}" />
-    </xacro:if>
-    <xacro:if value="${not add_gripper and not add_robotiq_arg85 and add_bio_gripper}">
+          ros2_control_plugin="${ros2_control_plugin}" dof="${dof}" hard_interface="${hard_interface}"
+          gripper_version="${gripper_version}" />
+      </xacro:unless>
+    </xacro:if>
+    <xacro:if value="${not add_gripper and add_bio_gripper}">
       <xacro:unless value="${robot_type == 'lite'}">
         <!-- Load BIO Gripper Model URDF -->
         <xacro:include filename="$(find xarm_description)/urdf/gripper/bio_gripper_macro.xacro" />
         <xacro:bio_gripper_macro prefix="${prefix}" attach_to="${prefix}link_eef"
-          ros2_control_plugin="${ros2_control_plugin}" dof="${dof}" hard_interface="${hard_interface}" />
-      </xacro:unless>
-    </xacro:if>
-    <xacro:if value="${not add_gripper and not add_robotiq_arg85 and not add_bio_gripper and add_vacuum_gripper}">
+          ros2_control_plugin="${ros2_control_plugin}" dof="${dof}" hard_interface="${hard_interface}"
+          gripper_version="${gripper_version}" />
+      </xacro:unless>
+    </xacro:if>
+    <xacro:if value="${not add_gripper and not add_bio_gripper and add_vacuum_gripper}">
       <xacro:if value="${robot_type == 'lite'}">
         <!-- Load Lite Vacuum Gripper Model URDF -->
@@ -258,5 +269,5 @@
       </xacro:unless>
     </xacro:if>
-    <xacro:if value="${not add_gripper and not add_robotiq_arg85 and not add_vacuum_gripper and add_other_geometry}">
+    <xacro:if value="${not add_gripper and not add_vacuum_gripper and add_other_geometry}">
       <!-- Load Other Model URDF -->
       <xacro:include filename="$(find xarm_description)/urdf/other/other_geometry.urdf.xacro" />
