Commit message: Update to xarm_ros2 jazzy 3dc2b5e (xarm_sdk v1.18.1)
Unmodified upstream xArm-Developer/xarm_ros2 jazzy branch, SDK submodule
included as plain files. This is the version built and tested with the
Lite6 on ROS 2 Jazzy.

Co-Authored-By: Claude Opus 5.5 <noreply@anthropic.com>

File: xarm_moveit_config/srdf/_lite6_macro.srdf.xacro (robot description, xacro)
@@ -10,5 +10,5 @@
   <!-- SUBGROUPS: Groups can also be formed by referencing to already defined group names -->
   <xacro:macro name="lite6_macro_srdf" params="prefix=''
-    add_gripper='false' add_vacuum_gripper='false' add_robotiq_arg85='false' add_other_geometry='false' ">
+    add_gripper='false' add_vacuum_gripper='false' add_other_geometry='false' ">
     <group name="${prefix}lite6">
       <joint name="${prefix}world_joint" />
@@ -25,12 +25,9 @@
         <joint name="${prefix}joint_tcp" />
       </xacro:if>
-      <xacro:if value="${not add_gripper and add_robotiq_arg85}">
-        <joint name="${prefix}robotiq_arg85_base_joint" />
-      </xacro:if>
-      <xacro:if value="${not add_gripper and not add_robotiq_arg85 and add_vacuum_gripper}">
+      <xacro:if value="${not add_gripper and add_vacuum_gripper}">
         <joint name="${prefix}vacuum_gripper_fix" />
         <joint name="${prefix}joint_tcp" />
       </xacro:if>
-      <xacro:if value="${not add_gripper and not add_robotiq_arg85 and not add_vacuum_gripper and add_other_geometry}">
+      <xacro:if value="${not add_gripper and not add_vacuum_gripper and add_other_geometry}">
         <joint name="${prefix}other_geometry_fix" />
         <joint name="${prefix}joint_tcp" />
@@ -48,40 +45,36 @@
     <!-- gripper -->
     <xacro:if value="${add_gripper}">
-      <!-- <group name="${prefix}lite_gripper">
-        <joint name="${prefix}gripper_fix" />
-        <joint name="${prefix}joint_tcp" />
-      </group> -->
+      <group name="${prefix}lite_gripper">
+        <link name="${prefix}uflite_gripper_link" />
+        <link name="${prefix}uflite_finger1" />
+        <link name="${prefix}uflite_finger2" />
+        <joint name="${prefix}finger_joint1" />
+      </group>
+      <group_state name="open" group="${prefix}lite_gripper">
+        <joint name="${prefix}finger_joint1" value="0.01" />
+      </group_state>
+      <group_state name="close" group="${prefix}lite_gripper">
+        <joint name="${prefix}finger_joint1" value="0" />
+      </group_state>
       <!-- END EFFECTOR, Purpose, Represent information about an end effector. -->
-      <!-- <end_effector name="${prefix}lite_gripper" parent_link="${prefix}link_tcp" group="${prefix}lite_gripper" /> -->
-      <passive_joint name="${prefix}gripper_fix" />
+      <end_effector name="${prefix}lite_gripper" parent_link="${prefix}link_tcp" group="${prefix}lite_gripper" />
+      <passive_joint name="${prefix}finger_joint2" />
       <!--PASSIVE JOINT, Purpose, this element is used to mark joints that are not actuated-->
       <!-- DISABLE COLLISIONS, By default it is assumed that any link of the robot could potentially come into collision with any other link in the robot. This tag disables collision checking between a specified pair of links. -->
-      <disable_collisions link1="${prefix}link5" link2="${prefix}uflite_gripper_link" reason="Never" />
-      <disable_collisions link1="${prefix}link6" link2="${prefix}uflite_gripper_link" reason="Never" />
-      <disable_collisions link1="${prefix}link_eef" link2="${prefix}uflite_gripper_link" reason="Adjacent" />
-    </xacro:if>
-    <xacro:if value="${not add_gripper and add_robotiq_arg85}">
-      <group name="${prefix}robotiq_arg85">
-        <joint name="${prefix}finger_joint" />
-      </group>
-      <end_effector name="${prefix}robotiq_arg85" parent_link="${prefix}link_eef" group="${prefix}robotiq_arg85" />
-      <passive_joint name="${prefix}left_inner_knuckle_joint" />
-      <passive_joint name="${prefix}left_inner_finger_joint" />
-      <passive_joint name="${prefix}right_inner_knuckle_joint" />
-      <passive_joint name="${prefix}right_inner_finger_joint" />
-      <passive_joint name="${prefix}right_outer_knuckle_joint" />
-      <disable_collisions link1="${prefix}link5" link2="${prefix}robotiq_85_base_link" reason="Never" />
-      <disable_collisions link1="${prefix}link6" link2="${prefix}robotiq_85_base_link" reason="Never" />
-      <disable_collisions link1="${prefix}link_eef" link2="${prefix}robotiq_85_base_link" reason="Adjacent" />
-      <disable_collisions link1="${prefix}robotiq_85_base_link" link2="${prefix}left_outer_knuckle" reason="Adjacent" />
-      <disable_collisions link1="${prefix}robotiq_85_base_link" link2="${prefix}left_inner_knuckle" reason="Adjacent" />
-      <disable_collisions link1="${prefix}robotiq_85_base_link" link2="${prefix}right_outer_knuckle" reason="Adjacent" />
-      <disable_collisions link1="${prefix}robotiq_85_base_link" link2="${prefix}right_inner_knuckle" reason="Adjacent" />
-      <disable_collisions link1="${prefix}left_outer_knuckle" link2="${prefix}left_outer_finger" reason="Adjacent" />
-      <disable_collisions link1="${prefix}left_inner_knuckle" link2="${prefix}left_inner_finger" reason="Adjacent" />
-      <disable_collisions link1="${prefix}right_outer_knuckle" link2="${prefix}right_outer_finger" reason="Adjacent" />
-      <disable_collisions link1="${prefix}right_inner_knuckle" link2="${prefix}right_inner_finger" reason="Adjacent" />
-      <disable_collisions link1="${prefix}left_outer_finger" link2="${prefix}left_inner_finger" reason="Default" />
-      <disable_collisions link1="${prefix}right_outer_finger" link2="${prefix}right_inner_finger" reason="Default" />
+      <disable_collisions link1="${prefix}uflite_gripper_link" link2="${prefix}uflite_finger1" reason="Adjacent" />
+      <disable_collisions link1="${prefix}uflite_gripper_link" link2="${prefix}uflite_finger2" reason="Adjacent" />
+      <disable_collisions link1="${prefix}uflite_finger1" link2="${prefix}uflite_finger2" reason="Never" />
+      <disable_collisions link1="${prefix}uflite_gripper_link" link2="${prefix}link4" reason="Never" />
+      <disable_collisions link1="${prefix}uflite_gripper_link" link2="${prefix}link5" reason="Never" />
+      <disable_collisions link1="${prefix}uflite_gripper_link" link2="${prefix}link6" reason="Adjacent" />
+      <disable_collisions link1="${prefix}uflite_gripper_link" link2="${prefix}link_eef" reason="Adjacent" />
+      <disable_collisions link1="${prefix}uflite_finger1" link2="${prefix}link4" reason="Never" />
+      <disable_collisions link1="${prefix}uflite_finger1" link2="${prefix}link5" reason="Never" />
+      <disable_collisions link1="${prefix}uflite_finger1" link2="${prefix}link6" reason="Never" />
+      <disable_collisions link1="${prefix}uflite_finger1" link2="${prefix}link_eef" reason="Never" />
+      <disable_collisions link1="${prefix}uflite_finger2" link2="${prefix}link4" reason="Never" />
+      <disable_collisions link1="${prefix}uflite_finger2" link2="${prefix}link5" reason="Never" />
+      <disable_collisions link1="${prefix}uflite_finger2" link2="${prefix}link6" reason="Never" />
+      <disable_collisions link1="${prefix}uflite_finger2" link2="${prefix}link_eef" reason="Never" />
     </xacro:if>
     <!-- vacuum gripper -->

File: xarm_moveit_config/srdf/xarm.srdf.xacro (robot description, xacro)
@@ -8,8 +8,7 @@
   <xacro:arg name="add_vacuum_gripper" default="false" />
   <xacro:arg name="add_bio_gripper" default="false" />
-  <xacro:arg name="add_robotiq_arg85" default="false" />
   <xacro:arg name="add_other_geometry" default="false" />
   <xacro:include filename="$(find xarm_moveit_config)/srdf/xarm_macro.srdf.xacro" />
   <xacro:xarm_macro_srdf prefix="$(arg prefix)" dof="$(arg dof)" robot_type="$(arg robot_type)"
-    add_gripper="$(arg add_gripper)" add_vacuum_gripper="$(arg add_vacuum_gripper)" add_bio_gripper="$(arg add_bio_gripper)" add_robotiq_arg85="$(arg add_robotiq_arg85)" add_other_geometry="$(arg add_other_geometry)" />
+    add_gripper="$(arg add_gripper)" add_vacuum_gripper="$(arg add_vacuum_gripper)" add_bio_gripper="$(arg add_bio_gripper)" add_other_geometry="$(arg add_other_geometry)" />
 </robot>

File: xarm_moveit_config/srdf/xarm_macro.srdf.xacro (robot description, xacro)
@@ -2,5 +2,5 @@
 <robot xmlns:xacro="http://wiki.ros.org/xacro" name="xarm_srdf">
   <xacro:macro name="xarm_macro_srdf" params="prefix:='' dof:=7 robot_type:='xarm'
-    add_gripper:='false' add_vacuum_gripper:='false' add_bio_gripper:='false' add_robotiq_arg85:='false' add_other_geometry:='false' ">
+    add_gripper:='false' add_vacuum_gripper:='false' add_bio_gripper:='false' add_other_geometry:='false' ">
     <xacro:if value="${dof == 5}">
       <xacro:include filename="$(find xarm_moveit_config)/srdf/_xarm5_macro.srdf.xacro" />
@@ -17,5 +17,5 @@
         <xacro:include filename="$(find xarm_moveit_config)/srdf/_lite6_macro.srdf.xacro" />
         <xacro:lite6_macro_srdf prefix="${prefix}"
-          add_gripper="${add_gripper}" add_vacuum_gripper="${add_vacuum_gripper}" add_robotiq_arg85="${add_robotiq_arg85}" add_other_geometry="${add_other_geometry}"  />
+          add_gripper="${add_gripper}" add_vacuum_gripper="${add_vacuum_gripper}" add_other_geometry="${add_other_geometry}"  />
       </xacro:if>
       <xacro:unless value="${robot_type == 'lite' or robot_type == 'uf850'}">
